Commit message: Harmonic
Signed-off-by: Juancams <jc.manzanares.serrano@gmail.com>

File: tiago_description/robots/tiago.urdf.xacro (robot description, xacro)
@@ -25,5 +25,5 @@
   <!-- pmb2, omni_base -->
   <xacro:arg name="base_type" default="pmb2"/>
-  <!-- no-laser, hokuyo, sick-551, sick-561, sick-571-->
+  no-laser, hokuyo, sick-551, sick-561, sick-571
   <xacro:arg name="laser_model" default="sick-571"/>
   <!-- false, true -->

File: tiago_description/ros2_control/ros2_control.urdf.xacro (robot description, xacro)
@@ -45,5 +45,5 @@
     <xacro:if value="${use_sim_time}">
       <gazebo>
-        <plugin filename="libgazebo_ros2_control.so" name="gazebo_ros2_control">
+        <plugin name="gz_ros2_control::GazeboSimROS2ControlPlugin" filename="gz_ros2_control-system">
           <parameters>$(find tiago_description)/ros2_control/gazebo_controller_manager_cfg.yaml</parameters>
         </plugin>
@@ -55,5 +55,5 @@
       <hardware>
         <xacro:if value="${use_sim_time}">
-          <plugin>gazebo_ros2_control/GazeboSystem</plugin>
+          <plugin>gz_ros2_control/GazeboSimSystem</plugin>
         <!-- IMU sensor (only in simulation)-->
         <xacro:ros2_control_imu name="base_imu_sensor"/>

File: tiago_description/urdf/arm/arm.urdf.xacro (robot description, xacro)
@@ -43,5 +43,5 @@
         <origin xyz="0.061191 -0.022397 ${reflect * -0.012835}" rpy="0.00000 0.00000 0.00000"/>
         <mass value="1.563428"/>
-        <inertia ixx="0.002471" ixy="${reflect * -0.001809}" ixz="-0.001202" iyy="0.006132" iyz="${reflect * 0.000494}" izz="0.006704"/>
+        <inertia ixx="0.002471" ixy="${-1 * -0.001809}" ixz="-0.001202" iyy="0.006132" iyz="${reflect * 0.000494}" izz="0.006704"/>
       </inertial>
       <!-- M90 module -->
@@ -49,5 +49,5 @@
         <origin xyz="0 0 0" rpy="0 0 0" />
         <geometry>
-          <mesh filename="package://tiago_description/meshes/arm/arm_1.stl" scale="1 ${-1 * tiago_dual} ${reflect}"/>
+          <mesh filename="file://$(find tiago_description)/meshes/arm/arm_1.stl" scale="1 ${-1 * tiago_dual} ${reflect}"/>
         </geometry>
         <material name="White"/>
@@ -56,5 +56,5 @@
         <origin xyz="0 0 0" rpy="0 0 0" />
         <geometry>
-          <mesh filename="package://tiago_description/meshes/arm/arm_1_collision.dae" scale="1 ${-1 * tiago_dual} ${reflect}"/>
+          <mesh filename="file://$(find tiago_description)/meshes/arm/arm_1_collision.dae" scale="1 ${-1 * tiago_dual} ${reflect}"/>
         </geometry>
       </collision>
@@ -81,5 +81,5 @@
         <origin xyz="0 0 0" rpy="${0 * deg_to_rad} ${0 * deg_to_rad} ${0 * deg_to_rad}" />
         <geometry>
-          <mesh filename="package://tiago_description/meshes/arm/arm_2.stl" scale="1 1 ${reflect}"/>
+          <mesh filename="file://$(find tiago_description)/meshes/arm/arm_2.stl" scale="1 1 ${reflect}"/>
         </geometry>
         <material name="DarkGrey" />
@@ -89,5 +89,5 @@
         <origin xyz="0 0 0" rpy="${0 * deg_to_rad} ${0 * deg_to_rad} ${0 * deg_to_rad}" />
         <geometry>
-          <mesh filename="package://tiago_description/meshes/arm/arm_2_collision.dae" scale="1 1 ${reflect}"/>
+          <mesh filename="file://$(find tiago_description)/meshes/arm/arm_2_collision.dae" scale="1 1 ${reflect}"/>
         </geometry>
       </collision>
@@ -113,5 +113,5 @@
         <origin xyz="0 0 0" rpy="0 0 0" />
         <geometry>
-          <mesh filename="package://tiago_description/meshes/arm/arm_3.stl" scale="1 1 ${reflect}"/>
+          <mesh filename="file://$(find tiago_description)/meshes/arm/arm_3.stl" scale="1 1 ${reflect}"/>
         </geometry>
         <material name="DarkGrey" />
@@ -120,5 +120,5 @@
         <origin xyz="0 0 0" rpy="0 0 0" />
         <geometry>
-          <mesh filename="package://tiago_description/meshes/arm/arm_3_collision.dae" scale="1 1 ${reflect}"/>
+          <mesh filename="file://$(find tiago_description)/meshes/arm/arm_3_collision.dae" scale="1 1 ${reflect}"/>
         </geometry>
       </collision>
@@ -145,5 +145,5 @@
         <origin xyz="0 0 0" rpy="0 0 0" />
         <geometry>
-          <mesh filename="package://tiago_description/meshes/arm/arm_4.stl" scale="${reflect} ${reflect} ${reflect}"/>
+          <mesh filename="file://$(find tiago_description)/meshes/arm/arm_4.stl" scale="${reflect} ${reflect} ${reflect}"/>
         </geometry>
         <material name="DarkGrey" />
@@ -152,5 +152,5 @@
         <origin xyz="0 0 0" rpy="0 0 0" />
         <geometry>
-          <mesh filename="package://tiago_description/meshes/arm/arm_4_collision.dae" scale="${reflect} ${reflect} ${reflect}"/>
+          <mesh filename="file://$(find tiago_description)/meshes/arm/arm_4_collision.dae" scale="${reflect} ${reflect} ${reflect}"/>
         </geometry>
       </collision>

File: tiago_description/urdf/arm/wrist.urdf.xacro (robot description, xacro)
@@ -50,5 +50,5 @@
         <origin xyz="0 0 0" rpy="0 0 0" />
         <geometry>
-          <mesh filename="package://tiago_description/meshes/arm/arm_5-${wrist_model}.stl" scale="${reflect} ${reflect} ${reflect}"/>
+          <mesh filename="file://$(find tiago_description)/meshes/arm/arm_5-${wrist_model}.stl" scale="${reflect} ${reflect} ${reflect}"/>
         </geometry>
         <material name="LightGrey" />
@@ -57,5 +57,5 @@
         <origin xyz="0 0 0" rpy="0 0 0" />
         <geometry>
-          <mesh filename="package://tiago_description/meshes/arm/arm_5_collision-${wrist_model}.dae" scale="${reflect} ${reflect} ${reflect}"/>
+          <mesh filename="file://$(find tiago_description)/meshes/arm/arm_5_collision-${wrist_model}.dae" scale="${reflect} ${reflect} ${reflect}"/>
         </geometry>
       </collision>
@@ -85,5 +85,5 @@
         <origin xyz="0 0 0" rpy="0 0 0" />
         <geometry>
-          <mesh filename="package://tiago_description/meshes/arm/arm_6-${wrist_model}.stl" scale="${reflect} 1 1"/>
+          <mesh filename="file://$(find tiago_description)/meshes/arm/arm_6-${wrist_model}.stl" scale="${reflect} 1 1"/>
         </geometry>
         <material name="LightGrey" />
@@ -92,5 +92,5 @@
         <origin xyz="0 0 0" rpy="0 0 0" />
         <geometry>
-          <mesh filename="package://tiago_description/meshes/arm/arm_6_collision-${wrist_model}.dae" scale="${reflect} 1 1"/>
+          <mesh filename="file://$(find tiago_description)/meshes/arm/arm_6_collision-${wrist_model}.dae" scale="${reflect} 1 1"/>
         </geometry>
       </collision>

File: tiago_description/urdf/head/head.urdf.xacro (robot description, xacro)
@@ -40,5 +40,5 @@
         <origin xyz="0 0 0" rpy="0 0 0"/>
         <geometry>
-          <mesh filename="package://tiago_description/meshes/head/head_1.stl" scale="1 1 1"/>
+          <mesh filename="file://$(find tiago_description)/meshes/head/head_1.stl" scale="1 1 1"/>
         </geometry>
         <material name="White" />
@@ -47,5 +47,5 @@
         <origin xyz="0.0 0 0" rpy="0 0 0.0" />
         <geometry>
-          <mesh filename="package://tiago_description/meshes/head/head_1_collision.dae" scale="1 1 1"/>
+          <mesh filename="file://$(find tiago_description)/meshes/head/head_1_collision.dae" scale="1 1 1"/>
         </geometry>
         <material name="White" />
@@ -80,5 +80,5 @@
         <origin xyz="0 0 0" rpy="0 0 0" />
         <geometry>
-          <mesh filename="package://tiago_description/meshes/head/head_2.stl" scale="1 1 1"/>
+          <mesh filename="file://$(find tiago_description)/meshes/head/head_2.stl" scale="1 1 1"/>
         </geometry>
         <material name="White" />
@@ -87,5 +87,5 @@
         <origin xyz="0 0 0" rpy="0 0 0" />
         <geometry>
-          <mesh filename="package://tiago_description/meshes/head/head_2_collision.dae" scale="1 1 1"/>
+          <mesh filename="file://$(find tiago_description)/meshes/head/head_2_collision.dae" scale="1 1 1"/>
         </geometry>
       </collision>

File: tiago_description/urdf/sensors/openni.gazebo.xacro (robot description, xacro)
@@ -40,8 +40,8 @@
           </distortion>
         </camera>
-        <plugin name="${name}_frame_controller" filename="libgazebo_ros_camera.so">
+        <!-- <plugin name="${name}_frame_controller" filename="libgazebo_ros_camera.so">
           <camera_name>${name}</camera_name>
           <ros>
-            <!-- <namespace>${name}</namespace>-->
+            <namespace>${name}</namespace>
             <remapping>${name}/image_raw:=${name}/rgb/image_raw</remapping>
             <remapping>${name}/camera_info:=${name}/rgb/camera_info</remapping>
@@ -53,5 +53,5 @@
           <min_depth>0.3</min_depth>
           <max_depth>8.0</max_depth>
-        </plugin>
+        </plugin> -->
       </sensor>
     </gazebo>

File: tiago_description/urdf/sensors/orbbec_astra.urdf.xacro (robot description, xacro)
@@ -35,5 +35,5 @@
         <origin xyz="0 0 0" rpy="0 0 0"/>
         <geometry>
-          <mesh filename="package://tiago_description/meshes/sensors/xtion_pro_live/xtion_pro_live.dae" />
+          <mesh filename="file://$(find tiago_description)/meshes/sensors/xtion_pro_live/xtion_pro_live.dae" />
         </geometry>
         <material name="Grey">

File: tiago_description/urdf/sensors/xtion_pro_live.urdf.xacro (robot description, xacro)
@@ -34,5 +34,5 @@
         <origin xyz="0 0 0" rpy="0 0 0"/>
         <geometry>
-          <mesh filename="package://tiago_description/meshes/sensors/xtion_pro_live/xtion_pro_live.dae" />
+          <mesh filename="file://$(find tiago_description)/meshes/sensors/xtion_pro_live/xtion_pro_live.dae" />
         </geometry>
         <material name="Grey">

File: tiago_description/urdf/torso/torso.urdf.xacro (robot description, xacro)
@@ -30,5 +30,5 @@
         <origin rpy="0 0 0" xyz="0 0 0" />
         <geometry>
-          <mesh filename="package://tiago_description/meshes/torso/torso_fix.stl" scale="1 1 1"/>
+          <mesh filename="file://$(find tiago_description)/meshes/torso/torso_fix.stl" scale="1 1 1"/>
         </geometry>
         <material name="LightGrey"/>
@@ -94,5 +94,5 @@
         <origin rpy="0 0 0" xyz="0 0 0" />
         <geometry>
-          <mesh filename="package://tiago_description/meshes/torso/torso_lift_with_arm.stl" scale="1 1 1"/>
+          <mesh filename="file://$(find tiago_description)/meshes/torso/torso_lift_with_arm.stl" scale="1 1 1"/>
         </geometry>
         <material name="White"/>
@@ -101,5 +101,5 @@
         <origin rpy="0 0 0" xyz="0 0 0" />
         <geometry>
-          <mesh filename="package://tiago_description/meshes/torso/torso_lift_collision_core.dae" scale="1 1 1"/>
+          <mesh filename="file://$(find tiago_description)/meshes/torso/torso_lift_collision_core.dae" scale="1 1 1"/>
         </geometry>
         <material name="LightGrey"/>
@@ -108,5 +108,5 @@
         <origin rpy="0 0 0" xyz="0 0 0" />
         <geometry>
-          <mesh filename="package://tiago_description/meshes/torso/torso_lift_collision_shoulder.dae" scale="1 1 1"/>
+          <mesh filename="file://$(find tiago_description)/meshes/torso/torso_lift_collision_shoulder.dae" scale="1 1 1"/>
         </geometry>
         <material name="LightGrey"/>
@@ -115,5 +115,5 @@
         <origin rpy="0 0 0" xyz="0 0 0" />
         <geometry>
-          <mesh filename="package://tiago_description/meshes/torso/torso_lift_collision_neck.dae" scale="1 1 1"/>
+          <mesh filename="file://$(find tiago_description)/meshes/torso/torso_lift_collision_neck.dae" scale="1 1 1"/>
         </geometry>
         <material name="LightGrey"/>
