Commit message: Changed torso range
Signed-off-by: Juancams <jc.manzanares.serrano@gmail.com>

File: tiago_description/urdf/torso/torso.urdf.xacro (robot description, xacro)
@@ -125,5 +125,5 @@
       <child link="${name}_lift_link" />
       <axis xyz="0 0 1" />
-      <limit effort="2000" lower="0" upper="0.35" velocity="${torso_max_vel}" />
+      <limit effort="2000" lower="-0.1" upper="0.35" velocity="${torso_max_vel}" />
       <calibration rising="0.0" />
       <dynamics damping="1000" />
